Commit message: refactor of packages

File: Software/ROS/src/dogbot_description/urdf/dogbot.xacro (robot description, xacro)
@@ -53,5 +53,5 @@
   </gazebo>
   <xacro:macro name="leg" params="prefix suffix reflectx reflecty">
-    <link name="${prefix}_${suffix}_roll">
+    <link name="${prefix}_${suffix}_hip">
       <visual>
         <origin xyz="0 0 0" rpy="${pi/2} 0 0" />
@@ -73,5 +73,5 @@
       <axis xyz="0 1 0" rpy="0 0 0" />
       <parent link="body"/>
-      <child link="${prefix}_${suffix}_roll"/>
+      <child link="${prefix}_${suffix}_hip"/>
       <origin xyz="${legoffset*reflectx} ${bodylen * reflecty/2} 0" rpy="0 0 ${-pi*(1-reflecty)/2}"/>
       <limit
@@ -111,5 +111,5 @@
     <joint name="${prefix}_${suffix}_pitch_joint" type="revolute">
       <axis xyz="0 1 0" rpy="0 0 0" />
-      <parent link="${prefix}_${suffix}_roll"/>
+      <parent link="${prefix}_${suffix}_hip"/>
       <child link="${prefix}_${suffix}_upperleg"/>
       <!--  rpy="0  ${pi * reflectx/2.3} ${pi *reflectx *reflecty /2} -->
@@ -178,5 +178,5 @@
         <hardwareInterface>hardware_interface/EffortJointInterface</hardwareInterface>
       </joint>
-      <actuator name="${prefix}_${suffix}_roll_actuator" >
+      <actuator name="${prefix}_${suffix}_roll_motor" >
         <hardwareInterface>hardware_interface/EffortJointInterface</hardwareInterface>
         <mechanicalReduction>1</mechanicalReduction>
@@ -188,5 +188,5 @@
         <hardwareInterface>hardware_interface/EffortJointInterface</hardwareInterface>
       </joint>
-      <actuator name="${prefix}_${suffix}_pitch_actuator" >
+      <actuator name="${prefix}_${suffix}_pitch_motor" >
         <hardwareInterface>hardware_interface/EffortJointInterface</hardwareInterface>
         <mechanicalReduction>1</mechanicalReduction>
@@ -198,5 +198,5 @@
         <hardwareInterface>hardware_interface/EffortJointInterface</hardwareInterface>
       </joint>
-      <actuator name="${prefix}_${suffix}_knee_actuator" >
+      <actuator name="${prefix}_${suffix}_knee_motor" >
         <hardwareInterface>hardware_interface/EffortJointInterface</hardwareInterface>
         <mechanicalReduction>1</mechanicalReduction>
